File: shunt.kicad_sch (KiCad schematic)
At the start: 33 parts, among them J1 Screw_Terminal_01x03, U1 INA219AxD

Commit message: Switch shunt footprint
The 2816 footprint is big enough to also mount all the smaller
resistors down to 1206 and allows munting the bigger 2816
resistors.
Parts:
- R2: footprint Project_Footprints:R_Dual_2512_1206_Handsolder -> Resistor_SMD:R_2816_7142Metric_Pad3.20x4.45mm_HandSolder
Changed lines of the file:
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@@
       (effects (font (size 1.27 1.27)) (justify left))
     )
-    (property "Footprint" "Project_Footprints:R_Dual_2512_1206_Handsolder" (id 2) (at 120.142 57.15 90)
+    (property "Footprint" "Resistor_SMD:R_2816_7142Metric_Pad3.20x4.45mm_HandSolder" (id 2) (at 120.142 57.15 90)
       (effects (font (size 1.27 1.27)) hide)
     )
